File: howland-current-source.kicad_sch (KiCad schematic)
At the start: 11 parts, among them J1 Conn_01x02

Commit message: Add PCB layout with routing complete
Parts:
- DA1, DA2: footprint howland_gost_footprints:OPA2277_DIP8 -> Package_DIP:DIP-8_W7.62mm
- J1: footprint (none) -> Connector_PinHeader_2.54mm:PinHeader_1x02_P2.54mm_Vertical
Changed lines of the file:
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@@
 			)
 		)
-		(property "Footprint" ""
+		(property "Footprint" "Connector_PinHeader_2.54mm:PinHeader_1x02_P2.54mm_Vertical"
 			(at 29.21 132.08 0)
 			(hide yes)
@@
 			)
 		)
-		(property "Footprint" "howland_gost_footprints:OPA2277_DIP8"
+		(property "Footprint" "Package_DIP:DIP-8_W7.62mm"
 			(at 111.76 81.28 0)
 			(hide yes)
@@
 			)
 		)
-		(property "Footprint" "howland_gost_footprints:OPA2277_DIP8"
+		(property "Footprint" "Package_DIP:DIP-8_W7.62mm"
 			(at 153.67 82.55 0)
 			(hide yes)
@@
 			)
 		)
-		(property "Footprint" "howland_gost_footprints:OPA2277_DIP8"
+		(property "Footprint" "Package_DIP:DIP-8_W7.62mm"
 			(at 245.11 83.82 0)
 			(hide yes)
@@
 			)
 		)
-		(property "Footprint" "howland_gost_footprints:OPA2277_DIP8"
+		(property "Footprint" "Package_DIP:DIP-8_W7.62mm"
 			(at 209.55 86.36 0)
 			(hide yes)
